File: Project/Loads2.kicad_sch (KiCad schematic)
At the start: 24 parts, among them J1 Load 0, J2 Load 1, J3 Load 2, J4 Load 3, J5 Load 4, J6 Load 7, J7 Load 6, J8 Load 5, K1 V23079C1103B301, K10 IMC03TS, K11 V23079C1103B301, K12 IMC03TS, K13 V23079C1103B301, K14 IMC03TS, K15 V23079C1103B301, K16 IMC03TS, K2 IMC03TS, K3 V23079C1103B301, K4 IMC03TS, K5 V23079C1103B301, K6 IMC03TS, K7 V23079C1103B301, K8 IMC03TS, K9 V23079C1103B301

Commit message: new 24 loads 25/10
Parts:
- renumbered J1 to J23, J2 to J24, J3 to J25, J4 to J26, J5 to J27, J7 to J29, J6 to J30, J8 to J31, K1 to K33, K3 to K34, K5 to K35, K7 to K36, K9 to K37, K2 to K38, K4 to K39, K6 to K40, K8 to K41, K10 to K42, K13 to K43, K15 to K44, K11 to K45, K14 to K46, K16 to K47, K12 to K48
Connections:
- net O1 renamed O33
- net O10 renamed O42
- net O11 renamed O43
- net O12 renamed O44
- net O13 renamed O45
- net O14 renamed O46
- net O15 renamed O47
- net O16 renamed O48
- net O2 renamed O34
- net O3 renamed O35
- net O4 renamed O36
- net O5 renamed O37
- net O6 renamed O38
- net O7 renamed O39
- net O8 renamed O40
- net O9 renamed O41
