File: Project/Loads-1.kicad_sch (KiCad schematic)
At the start: 24 parts, among them J22 Load 0, J23 Load 1, J24 Load 2, J25 Load 3, J26 Load 4, J27 Load 6, J28 Load 7, J29 Load 5, K33 V23079C1103B301, K34 V23079C1103B301, K35 V23079C1103B301, K36 V23079C1103B301, K37 V23079C1103B301, K38 IMC03TS, K39 IMC03TS, K40 IMC03TS, K41 IMC03TS, K42 IMC03TS, K43 V23079C1103B301, K44 V23079C1103B301, K45 V23079C1103B301, K46 IMC03TS, K47 IMC03TS, K48 IMC03TS

Commit message: new 08/11
Parts:
- renumbered K33 to K1, K42 to K10, K43 to K11, K44 to K12, K45 to K13, K46 to K14, K47 to K15, K48 to K16, K34 to K2, K35 to K3, K36 to K4, K37 to K5, K38 to K6, K39 to K7, K40 to K8, K41 to K9, J22 to Load_0, J23 to Load_1, J24 to Load_2, J25 to Load_3, J26 to Load_4, J29 to Load_5, J27 to Load_6, J28 to Load_7
Connections:
- net O33 renamed O1
- net O34 renamed O2
- net O35 renamed O3
- net O36 renamed O4
- net O37 renamed O5
- net O38 renamed O6
- net O39 renamed O7
- net O40 renamed O8
- net O41 renamed O9
- net O42 renamed O10
- net O43 renamed O11
- net O44 renamed O12
- net O45 renamed O13
- net O46 renamed O14
- net O47 renamed O15
- net O48 renamed O16
