File: Project/Loads-2.kicad_sch (KiCad schematic)
At the start: 24 parts, among them J22 Load 0, J23 Load 1, J24 Load 2, J25 Load 3, J26 Load 4, J27 Load 6, J28 Load 7, J29 Load 5, K33 V23079C1103B301, K34 V23079C1103B301, K35 V23079C1103B301, K36 V23079C1103B301, K37 V23079C1103B301, K38 IMC03TS, K39 IMC03TS, K40 IMC03TS, K41 IMC03TS, K42 IMC03TS, K43 V23079C1103B301, K44 V23079C1103B301, K45 V23079C1103B301, K46 IMC03TS, K47 IMC03TS, K48 IMC03TS

Commit message: new 08/11
Parts:
- Load_10: renamed from J24; value Load 2 -> Load 10
- Load_11: renamed from J25; value Load 3 -> Load 11
- Load_12: renamed from J26; value Load 4 -> Load 12
- Load_13: renamed from J29; value Load 5 -> Load 13
- Load_14: renamed from J27; value Load 6 -> Load 14
- Load_15: renamed from J28; value Load 7 -> Load 15
- Load_8: renamed from J22; value Load 0 -> Load 8
- Load_9: renamed from J23; value Load 1 -> Load 9
- renumbered K33 to K17, K34 to K18, K35 to K19, K36 to K20, K37 to K21, K38 to K22, K39 to K23, K40 to K24, K41 to K25, K42 to K26, K43 to K27, K44 to K28, K45 to K29, K46 to K30, K47 to K31, K48 to K32
Connections:
- net O33 renamed O17
- net O34 renamed O18
- net O35 renamed O19
- net O36 renamed O20
- net O37 renamed O21
- net O38 renamed O22
- net O39 renamed O23
- net O40 renamed O24
- net O41 renamed O25
- net O42 renamed O26
- net O43 renamed O27
- net O44 renamed O28
- net O45 renamed O29
- net O46 renamed O30
- net O47 renamed O31
- net O48 renamed O32
