File: Project/Loads-3.kicad_sch (KiCad schematic)
At the start: 24 parts, among them J22 Load 0, J23 Load 1, J24 Load 2, J25 Load 3, J26 Load 4, J27 Load 6, J28 Load 7, J29 Load 5, K33 V23079C1103B301, K34 V23079C1103B301, K35 V23079C1103B301, K36 V23079C1103B301, K37 V23079C1103B301, K38 IMC03TS, K39 IMC03TS, K40 IMC03TS, K41 IMC03TS, K42 IMC03TS, K43 V23079C1103B301, K44 V23079C1103B301, K45 V23079C1103B301, K46 IMC03TS, K47 IMC03TS, K48 IMC03TS

Commit message: new 08/11
Parts:
- Load_16: renamed from J22; value Load 0 -> Load 16
- Load_17: renamed from J23; value Load 1 -> Load 17
- Load_18: renamed from J24; value Load 2 -> Load 18
- Load_19: renamed from J25; value Load 3 -> Load 19
- Load_20: renamed from J26; value Load 4 -> Load 20
- Load_21: renamed from J29; value Load 5 -> Load 21
- Load_22: renamed from J27; value Load 6 -> Load 22
- Load_23: renamed from J28; value Load 7 -> Load 23
Changed lines of the file:
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@@
 		(on_board yes)
 		(dnp no)
-		(property "Reference" "J27"
+		(property "Reference" "Load_22"
 			(at 260.858 60.706 0)
 			(effects
@@
 			)
 		)
-		(property "Value" "Load 6"
+		(property "Value" "Load 22"
 			(at 252.222 72.644 0)
 			(effects
@@
 			(project "load_automatisation"
 				(path "/e193aeee-7d8e-4a61-b3f1-51249c7839f9/9a4a53da-5e5a-4867-b392-518dc37283c5/ac2d2ff3-bffa-4c87-aa18-e5cd5cb143e2"
-					(reference "J27")
+					(reference "Load_22")
 					(unit 1)
 				)
@@
 		(on_board yes)
 		(dnp no)
-		(property "Reference" "J24"
+		(property "Reference" "Load_18"
 			(at 121.158 93.726 0)
 			(effects
@@
 			)
 		)
-		(property "Value" "Load 2"
+		(property "Value" "Load 18"
 			(at 112.522 105.664 0)
 			(effects
@@
 			(project "load_automatisation"
 				(path "/e193aeee-7d8e-4a61-b3f1-51249c7839f9/9a4a53da-5e5a-4867-b392-518dc37283c5/ac2d2ff3-bffa-4c87-aa18-e5cd5cb143e2"
-					(reference "J24")
+					(reference "Load_18")
 					(unit 1)
 				)
@@
 		(on_board yes)
 		(dnp no)
-		(property "Reference" "J26"
+		(property "Reference" "Load_20"
 			(at 123.698 166.116 0)
 			(effects
@@
 			)
 		)
-		(property "Value" "Load 4"
+		(property "Value" "Load 20"
 			(at 115.062 178.054 0)
 			(effects
@@
 			(project "load_automatisation"
 				(path "/e193aeee-7d8e-4a61-b3f1-51249c7839f9/9a4a53da-5e5a-4867-b392-518dc37283c5/ac2d2ff3-bffa-4c87-aa18-e5cd5cb143e2"
-					(reference "J26")
+					(reference "Load_20")
 					(unit 1)
 				)
@@
 		(on_board yes)
 		(dnp no)
-		(property "Reference" "J28"
+		(property "Reference" "Load_23"
 			(at 260.858 100.076 0)
 			(effects
@@
 			)
 		)
-		(property "Value" "Load 7"
+		(property "Value" "Load 23"
 			(at 252.222 112.014 0)
 			(effects
@@
 			(project "load_automatisation"
 				(path "/e193aeee-7d8e-4a61-b3f1-51249c7839f9/9a4a53da-5e5a-4867-b392-518dc37283c5/ac2d2ff3-bffa-4c87-aa18-e5cd5cb143e2"
-					(reference "J28")
+					(reference "Load_23")
 					(unit 1)
 				)
@@
 		(on_board yes)
 		(dnp no)
-		(property "Reference" "J29"
+		(property "Reference" "Load_21"
 			(at 263.398 20.066 0)
 			(effects
@@
 			)
 		)
-		(property "Value" "Load 5"
+		(property "Value" "Load 21"
 			(at 254.762 32.004 0)
 			(effects
@@
 			(project "load_automatisation"
 				(path "/e193aeee-7d8e-4a61-b3f1-51249c7839f9/9a4a53da-5e5a-4867-b392-518dc37283c5/ac2d2ff3-bffa-4c87-aa18-e5cd5cb143e2"
-					(reference "J29")
+					(reference "Load_21")
 					(unit 1)
 				)
@@
 		(on_board yes)
 		(dnp no)
-		(property "Reference" "J22"
+		(property "Reference" "Load_16"
 			(at 121.158 17.526 0)
 			(effects
@@
 			)
 		)
-		(property "Value" "Load 0"
+		(property "Value" "Load 16"
 			(at 112.522 29.464 0)
 			(effects
@@
 			(project "load_automatisation"
 				(path "/e193aeee-7d8e-4a61-b3f1-51249c7839f9/9a4a53da-5e5a-4867-b392-518dc37283c5/ac2d2ff3-bffa-4c87-aa18-e5cd5cb143e2"
-					(reference "J22")
+					(reference "Load_16")
 					(unit 1)
 				)
@@
 		(on_board yes)
 		(dnp no)
-		(property "Reference" "J25"
+		(property "Reference" "Load_19"
 			(at 121.158 129.286 0)
 			(effects
@@
 			)
 		)
-		(property "Value" "Load 3"
+		(property "Value" "Load 19"
 			(at 112.522 141.224 0)
 			(effects
@@
 			(project "load_automatisation"
 				(path "/e193aeee-7d8e-4a61-b3f1-51249c7839f9/9a4a53da-5e5a-4867-b392-518dc37283c5/ac2d2ff3-bffa-4c87-aa18-e5cd5cb143e2"
-					(reference "J25")
+					(reference "Load_19")
 					(unit 1)
 				)
@@
 		(on_board yes)
 		(dnp no)
-		(property "Reference" "J23"
+		(property "Reference" "Load_17"
 			(at 121.158 56.896 0)
 			(effects
@@
 			)
 		)
-		(property "Value" "Load 1"
+		(property "Value" "Load 17"
 			(at 112.522 68.834 0)
 			(effects
@@
 			(project "load_automatisation"
 				(path "/e193aeee-7d8e-4a61-b3f1-51249c7839f9/9a4a53da-5e5a-4867-b392-518dc37283c5/ac2d2ff3-bffa-4c87-aa18-e5cd5cb143e2"
-					(reference "J23")
+					(reference "Load_17")
 					(unit 1)
 				)
