File: Project/Loads.kicad_sch (KiCad schematic)
At the start: 24 parts, among them J1 Load 0, J2 Load 1, J3 Load 2, J4 Load 3, J5 Load 4, J6 Load 7, J7 Load 6, J8 Load 5, K1 V23079C1103B301, K10 IMC03TS, K11 V23079C1103B301, K12 IMC03TS, K13 V23079C1103B301, K14 IMC03TS, K15 V23079C1103B301, K16 IMC03TS, K2 IMC03TS, K3 V23079C1103B301, K4 IMC03TS, K5 V23079C1103B301, K6 IMC03TS, K7 V23079C1103B301, K8 IMC03TS, K9 V23079C1103B301

Commit message: new 08/11
Parts:
- renumbered J7 to J6, J6 to J7, K13 to K11, K15 to K12, K11 to K13, K16 to K15, K12 to K16, K3 to K2, K5 to K3, K7 to K4, K9 to K5, K2 to K6, K4 to K7, K6 to K8, K8 to K9
