File: Project/Loads1.kicad_sch (KiCad schematic)
At the start: 24 parts, among them J1 Load 0, J2 Load 1, J3 Load 2, J4 Load 3, J5 Load 4, J6 Load 7, J7 Load 6, J8 Load 5, K1 V23079C1103B301, K10 IMC03TS, K11 V23079C1103B301, K12 IMC03TS, K13 V23079C1103B301, K14 IMC03TS, K15 V23079C1103B301, K16 IMC03TS, K2 IMC03TS, K3 V23079C1103B301, K4 IMC03TS, K5 V23079C1103B301, K6 IMC03TS, K7 V23079C1103B301, K8 IMC03TS, K9 V23079C1103B301

Commit message: new 24 loads 25/10
Parts:
- renumbered J1 to J14, J2 to J15, J3 to J16, J4 to J17, J5 to J18, J7 to J20, J6 to J21, J8 to J22, K1 to K17, K3 to K18, K5 to K19, K7 to K20, K9 to K21, K2 to K22, K4 to K23, K6 to K24, K8 to K25, K10 to K26, K13 to K27, K15 to K28, K11 to K29, K14 to K30, K16 to K31, K12 to K32
Connections:
- net O1 renamed O17
- net O10 renamed O26
- net O11 renamed O27
- net O12 renamed O28
- net O13 renamed O29
- net O14 renamed O30
- net O15 renamed O31
- net O16 renamed O32
- net O2 renamed O18
- net O3 renamed O19
- net O4 renamed O20
- net O5 renamed O21
- net O6 renamed O22
- net O7 renamed O23
- net O8 renamed O24
- net O9 renamed O25

Commit message: new 08/11
Parts:
- renumbered J14 to J10, J15 to J14, J16 to J15, J17 to J16, J18 to J17, J20 to J18, J21 to J20, J22 to J21
