File: Project/load_automatisation.kicad_pcb (KiCad board)
At the start: 2 copper layers, 49 parts, among them IC1 DRDC3105F-7, IC10 DRDC3105F-7, IC11 DRDC3105F-7, IC12 DRDC3105F-7, IC13 DRDC3105F-7, IC14 DRDC3105F-7, IC15 DRDC3105F-7, IC16 DRDC3105F-7, IC17 DRDC3105F-7, IC2 DRDC3105F-7, IC3 MC74VHC138DR2G, IC4 DRDC3105F-7, IC5 DRDC3105F-7, IC6 DRDC3105F-7, IC7 DRDC3105F-7, IC8 DRDC3105F-7, IC9 DRDC3105F-7, J1 Conn_01x03_Socket, J10 DadConnector, J11 TENG, J2 Conn_01x03_Socket, J3 Conn_01x03_Socket, J4 Conn_01x03_Socket, J5 Conn_01x03_Socket, J6 Conn_01x03_Socket, J7 Conn_01x03_Socket, J8 Conn_01x03_Socket, J9 PowerIn, K1 IMC03TS, K10 IMC03TS, K11 IMC03TS, K12 IMC03TS, K13 IMC03TS, K14 IMC03TS, K15 IMC03TS, K16 IMC03TS, K2 V23079C1103B301, K3 V23079C1103B301, K4 V23079C1103B301, K5 V23079C1103B301, K6 V23079C1103B301, K7 V23079C1103B301, K8 V23079C1103B301, K9 V23079C1103B301, U1 AMS1117-5.0

Commit message: new schematic
Parts:
- IC1, IC10, IC11, IC12, IC13, IC14, IC15, IC16, IC17, IC2, IC4, IC5, IC6, IC7, IC8, IC9: footprint SamacSys_Parts:SOT96P240X110-3N -> Library:SOT96P240X110-3N
- IC3: footprint SamacSys_Parts:SOIC127P600X175-16N -> Library:SOIC127P600X175-16N
- J1: value Conn_01x03_Socket -> Load 0
- J2: value Conn_01x03_Socket -> Load 1
- J3: value Conn_01x03_Socket -> Load 2
- J4: value Conn_01x03_Socket -> Load 3
- J5: value Conn_01x03_Socket -> Load 4
- J6: value Conn_01x03_Socket -> Load 7
- J7: value Conn_01x03_Socket -> Load 6
- J8: value Conn_01x03_Socket -> Load 5
- K1, K11, K13, K15: value IMC03TS -> V23079C1103B301; footprint SamacSys_Parts:IMC03TS -> Library:V23079A1001B301
- K10, K12, K14, K16: footprint SamacSys_Parts:IMC03TS -> Library:IMC03TS
- K2, K4, K6, K8: value V23079C1103B301 -> IMC03TS; footprint SamacSys_Parts:V23079A1001B301 -> Library:IMC03TS
- K3, K5, K7, K9: footprint SamacSys_Parts:V23079A1001B301 -> Library:V23079A1001B301
- moved K16 166.6 mm to (253.9, 121.4), turned to 0 degrees
- moved IC16 137.2 mm to (245.5, 128.3), turned to 0 degrees
- moved K15 134.8 mm to (259.9, 109.2), turned to 0 degrees
- moved K12 133.1 mm to (228.2, 51.0), turned to 0 degrees
- moved IC17 133.0 mm to (245.4, 112.7), turned to 0 degrees
- moved J6 122.3 mm to (247.8, 96.2)
- moved IC13 105.8 mm to (205.3, 62.0), turned to 0 degrees
- moved J9 101.7 mm to (58.3, 139.9), turned to 90 degrees
- moved J8 101.6 mm to (199.0, 29.9)
- moved IC12 99.9 mm to (224.6, 63.2), turned to 0 degrees
- moved J5 98.1 mm to (119.6, 126.1), turned to 90 degrees
- moved K1 96.5 mm to (48.3, 73.8)
- moved K11 94.8 mm to (211.3, 49.5)
- moved IC2 93.6 mm to (41.6, 82.7)
- moved K13 88.3 mm to (194.3, 120.0), turned to 0 degrees
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Connections:
- net V_OUT_1 renamed Net-(IC1-OUT)
- net V_OUT_11 renamed Net-(IC9-OUT)
- net V_OUT_5 renamed Net-(IC4-OUT)
- net Y6 renamed /Y6
- net Y7 renamed /Y7
- IC1 pad 1: Y0 -> /Y0
- IC10 pad 1: Y0 -> /Y4
- IC10 pad 3: V_OUT_2 -> Net-(IC10-OUT)
- IC11 pad 1: Y1 -> /Y4
- IC11 pad 3: V_OUT_4 -> Net-(IC11-OUT)
- IC12 pad 1: Y2 -> /Y5
- IC12 pad 3: V_OUT_6 -> Net-(IC12-OUT)
- IC13 pad 1: Y5 -> /Y5
- IC13 pad 3: V_OUT_12 -> Net-(IC13-OUT)
- IC14 pad 3: V_OUT_13 -> Net-(IC14-OUT)
- IC15 pad 3: V_OUT_14 -> Net-(IC15-OUT)
- IC16 pad 3: V_OUT_15 -> Net-(IC16-OUT)
- IC17 pad 3: V_OUT_16 -> Net-(IC17-OUT)
- IC2 pad 1: Y1 -> /Y0
- IC2 pad 3: V_OUT_3 -> Net-(IC2-OUT)
- IC3 pad 1: DAQ_Output_1.0 -> /Din0
- IC3 pad 10: Y5 -> /Y5
- IC3 pad 11: Y4 -> /Y4
- IC3 pad 12: Y3 -> /Y3
- IC3 pad 13: Y2 -> /Y2
- IC3 pad 14: Y1 -> /Y1
- IC3 pad 15: Y0 -> /Y0
- IC3 pad 16: +5V -> VCC
- IC3 pad 2: DAQ_Output_1.1 -> /Din1
- IC3 pad 3: DAQ_Output_1.2 -> /Din2
- IC3 pad 4: DAQ_Output_1.3 -> /Din3
- IC3 pad 5: DAQ_Output_1.4 -> /Din4
- IC3 pad 6: DAQ_Output_1.5 -> /Din5
- IC4 pad 1: Y2 -> /Y1
- IC5 pad 1: Y3 -> /Y1
- IC5 pad 3: V_OUT_7 -> Net-(IC5-OUT)
- IC6 pad 1: Y3 -> /Y2
- IC6 pad 3: V_OUT_8 -> Net-(IC6-OUT)
- IC7 pad 1: Y4 -> /Y2
- IC7 pad 3: V_OUT_9 -> Net-(IC7-OUT)
- IC8 pad 1: Y4 -> /Y3
- IC8 pad 3: V_OUT_10 -> Net-(IC8-OUT)
- IC9 pad 1: Y5 -> /Y3
- K1 pad 1: V_OUT_2 -> Net-(IC2-OUT)
- K1 pad 3: Rc_1 -> unconnected-(K1-NC_1-Pad3)
- K1 pad 5: DAQ - -> /Teng+
- K1 pad 8: GND -> /Vsense
- K10 pad 1: V_OUT_4 -> Net-(IC10-OUT)
- K10 pad 3: Rc_2 -> /Loads/Rc_4
- K10 pad 5: DAQ - -> /Teng-
- K11 pad 1: V_OUT_6 -> Net-(IC13-OUT)
- K11 pad 3: Rc_3 -> unconnected-(K11-NC_1-Pad3)
- K11 pad 5: DAQ - -> /Teng+
- K11 pad 8: GND -> /Vsense
- K12 pad 1: V_OUT_16 -> Net-(IC12-OUT)
- K12 pad 3: Rc_8 -> /Loads/Rc_5
- K12 pad 5: DAQ - -> /Teng-
- K13 pad 1: V_OUT_10 -> Net-(IC15-OUT)
- K13 pad 3: Rc_5 -> unconnected-(K13-NC_1-Pad3)
- K13 pad 5: DAQ - -> /Teng+
- K13 pad 8: GND -> /Vsense
- K14 pad 1: V_OUT_14 -> Net-(IC14-OUT)
- K14 pad 3: Rc_7 -> /Loads/Rc_6
- K14 pad 5: DAQ - -> /Teng-
- K15 pad 1: V_OUT_8 -> Net-(IC17-OUT)
- K15 pad 3: Rc_4 -> unconnected-(K15-NC_1-Pad3)
- K15 pad 5: DAQ - -> /Teng+
- K15 pad 8: GND -> /Vsense
- K16 pad 1: V_OUT_12 -> Net-(IC16-OUT)
- K16 pad 3: Rc_6 -> /Loads/Rc_7
- K16 pad 5: DAQ - -> /Teng-
- K2 pad 3: unconnected-(K2-NC_1-Pad3) -> /Loads/Ra_0
- K2 pad 5: TENG + -> /Teng-
- K2 pad 8: DAQ + -> GND
- K3 pad 1: V_OUT_3 -> Net-(IC5-OUT)
- K3 pad 4: Ra_2 -> /Loads/Rb_1
- K3 pad 5: TENG + -> /Teng+
- K3 pad 8: DAQ + -> /Vsense
- K3 pad 9: Rb_2 -> /Loads/Ra_1
- K4 pad 3: unconnected-(K4-NC_1-Pad3) -> /Loads/Rc_1
- K4 pad 5: TENG + -> /Teng-
- K4 pad 8: DAQ + -> GND
- K5 pad 1: V_OUT_7 -> Net-(IC7-OUT)
- K5 pad 4: Ra_4 -> /Loads/Rb_2
- K5 pad 5: TENG + -> /Teng+
- K5 pad 8: DAQ + -> /Vsense
- K5 pad 9: Rb_4 -> /Loads/Ra_2
- K6 pad 1: V_OUT_9 -> Net-(IC6-OUT)
- K6 pad 3: unconnected-(K6-NC_1-Pad3) -> /Loads/Rc_2
- K6 pad 5: TENG + -> /Teng-
- K6 pad 8: DAQ + -> GND
- K7 pad 4: Ra_6 -> /Loads/Rb_3
- K7 pad 5: TENG + -> /Teng+
- K7 pad 8: DAQ + -> /Vsense
- K7 pad 9: Rb_6 -> /Loads/Ra_3
- K8 pad 1: V_OUT_13 -> Net-(IC8-OUT)
- K8 pad 3: unconnected-(K8-NC_1-Pad3) -> /Loads/Rc_3
- K8 pad 5: TENG + -> /Teng-
- K8 pad 8: DAQ + -> GND
- K9 pad 1: V_OUT_15 -> Net-(IC11-OUT)
- K9 pad 4: Ra_8 -> /Loads/Rb_4
- K9 pad 5: TENG + -> /Teng+
- K9 pad 8: DAQ + -> /Vsense
- K9 pad 9: Rb_8 -> /Loads/Ra_4

Commit message: update schematic
Parts:
- added J12: Load 0, Connector_PinHeader_2.54mm:PinHeader_1x03_P2.54mm_Horizontal, F.Cu at (-65.8, 142.5)
- added J13: DIN41612_02x05_AB_EvenPins, Connector_PinSocket_2.54mm:PinSocket_2x05_P2.54mm_Vertical, F.Cu at (43.3, 128.9)
- added JP1: Jumper_3_Bridged12, Connector_PinHeader_2.54mm:PinHeader_1x03_P2.54mm_Vertical, F.Cu at (32.0, 73.5)
- added R2: R, Resistor_SMD:R_0805_2012Metric, F.Cu at (-54.0, 145.0)
- added R3: R, Resistor_SMD:R_0805_2012Metric, F.Cu at (-59.0, 145.1)
- added R4: R, Resistor_SMD:R_0805_2012Metric, F.Cu at (-58.9, 141.4)
- added R5: R, Resistor_THT:R_Axial_DIN0614_L14.3mm_D5.7mm_P20.32mm_Horizontal, F.Cu at (-47.7, 128.5)
- added R6: R, Resistor_SMD:R_0805_2012Metric, F.Cu at (-59.0, 137.5)
- added R7: R, Resistor_SMD:R_0805_2012Metric, F.Cu at (-59.0, 133.7)
- moved R1 50.1 mm to (30.0, 128.0)
- moved J9 28.7 mm to (39.2, 161.3)
- moved K4 20.2 mm to (80.0, 67.0), turned to 90 degrees
- moved IC4 13.5 mm to (89.0, 71.0), turned to 180 degrees
- moved IC5 12.3 mm to (89.0, 88.0), turned to 180 degrees
- moved K3 10.5 mm to (80.0, 82.0), turned to 90 degrees
- moved J10 9.99 mm to (25.1, 95.1)
- moved J2 9.38 mm to (80.5, 57.0), turned to 180 degrees
- moved J11 7.81 mm to (25.3, 57.2)
- moved K5 5.15 mm to (123.4, 71.5)
- moved IC6 5.14 mm to (135.7, 81.7)
- moved J3 5.00 mm to (128.6, 61.9)
- moved IC7 4.46 mm to (118.5, 82.0)
- moved IC1 3.98 mm to (62.6, 79.7), turned to 90 degrees
- moved IC2 3.67 mm to (44.2, 80.1), turned to 90 degrees
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Connections:
- J11 pad 2: /Teng- -> /TengN
Routing:
- net /Din2: track 0.00 -> 31.7 mm
- net /Din1: track 0.00 -> 31.0 mm
- net /Din0: track 0.00 -> 30.5 mm
- net /Loads/Ra_0: track 0.00 -> 17.4 mm
- net /Loads/Rb_0: track 0.00 -> 16.1 mm
- net /Loads/Rc_0: track 0.00 -> 9.56 mm
Other:
- board outline added: 143.5 x 116.5 mm

Commit message: new 24 loads 25/10
Parts:
- removed IC11, IC12, IC13, IC14, IC15, IC16, IC17: DRDC3105F-7, Library:SOT96P240X110-3N
- removed J13: DIN41612_02x05_AB_EvenPins, Connector_PinSocket_2.54mm:PinSocket_2x05_P2.54mm_Vertical
- removed JP1: Jumper_3_Bridged12, Connector_PinHeader_2.54mm:PinHeader_1x03_P2.54mm_Vertical
- removed R7: R, Resistor_SMD:R_0805_2012Metric
- added C4: 100nF, Capacitor_SMD:C_0805_2012Metric, F.Cu at (25.5, 87.0)
- added C5: 100nF, Capacitor_SMD:C_0805_2012Metric, F.Cu at (86.0, 74.5)
- added C6: 100nF, Capacitor_SMD:C_0805_2012Metric, F.Cu at (74.5, 105.0)
- added J14: Load 0, Connector_PinHeader_2.54mm:PinHeader_1x03_P2.54mm_Vertical, F.Cu at (214.6, 20.3)
- added J15: Load 1, Connector_PinHeader_2.54mm:PinHeader_1x03_P2.54mm_Vertical, F.Cu at (243.8, 20.3)
- added J16: Load 2, Connector_PinHeader_2.54mm:PinHeader_1x03_P2.54mm_Vertical, F.Cu at (270.5, 20.3)
- added J17: Load 3, Connector_PinHeader_2.54mm:PinHeader_1x03_P2.54mm_Vertical, F.Cu at (303.5, 20.3)
- added J18: Load 4, Connector_PinHeader_2.54mm:PinHeader_1x03_P2.54mm_Vertical, F.Cu at (102.9, 20.3)
- added J19: DaqConnector, SamacSys_Parts:231339001000, F.Cu at (26.5, 148.4)
- added J20: Load 6, Connector_PinHeader_2.54mm:PinHeader_1x03_P2.54mm_Vertical, F.Cu at (161.3, 20.3)
- added J21: Load 7, Connector_PinHeader_2.54mm:PinHeader_1x03_P2.54mm_Vertical, F.Cu at (189.2, 20.3)
- added J22: Load 5, Connector_PinHeader_2.54mm:PinHeader_1x03_P2.54mm_Vertical, F.Cu at (132.1, 20.3)
- added J23: Load 0, Connector_PinHeader_2.54mm:PinHeader_1x03_P2.54mm_Vertical, F.Cu at (319.3, 139.7)
- added J24: Load 1, Connector_PinHeader_2.54mm:PinHeader_1x03_P2.54mm_Vertical, F.Cu at (318.0, 118.1)
- added J25: Load 2, Connector_PinHeader_2.54mm:PinHeader_1x03_P2.54mm_Vertical, F.Cu at (318.0, 95.2)
- added J26: Load 3, Connector_PinHeader_2.54mm:PinHeader_1x03_P2.54mm_Vertical, F.Cu at (318.0, 72.3)
- added J27: Load 4, Connector_PinHeader_2.54mm:PinHeader_1x03_P2.54mm_Vertical, F.Cu at (294.1, 246.0)
- added J29: Load 6, Connector_PinHeader_2.54mm:PinHeader_1x03_P2.54mm_Vertical, F.Cu at (294.1, 193.9)
- added J30: Load 7, Connector_PinHeader_2.54mm:PinHeader_1x03_P2.54mm_Vertical, F.Cu at (295.4, 164.7)
- added J31: Load 5, Connector_PinHeader_2.54mm:PinHeader_1x03_P2.54mm_Vertical, F.Cu at (294.1, 218.1)
- added JP2: Jumper_3_Bridged12, Jumper:SolderJumper-3_P1.3mm_Bridged2Bar12_Pad1.0x1.5mm_NumberLabels, F.Cu at (51.2, 92.5)
- added K17: V23079C1103B301, SamacSys_Parts:V23079A1001B301, F.Cu at (222.3, 48.2)
- added K18: V23079C1103B301, SamacSys_Parts:V23079A1001B301, F.Cu at (250.2, 48.2)
- added K19: V23079C1103B301, SamacSys_Parts:V23079A1001B301, F.Cu at (278.1, 49.5)
- added K20: V23079C1103B301, SamacSys_Parts:V23079A1001B301, F.Cu at (312.4, 48.2)
- added K21: V23079C1103B301, SamacSys_Parts:V23079A1001B301, F.Cu at (108.0, 48.2)
- added K22: IMC03TS, SamacSys_Parts:IMC03TS, F.Cu at (208.5, 48.2)
- added K23: IMC03TS, SamacSys_Parts:IMC03TS, F.Cu at (237.7, 48.9)
- added K24: IMC03TS, SamacSys_Parts:IMC03TS, F.Cu at (264.4, 49.5)
- added K25: IMC03TS, SamacSys_Parts:IMC03TS, F.Cu at (296.1, 49.5)
- added K26: IMC03TS, SamacSys_Parts:IMC03TS, F.Cu at (94.0, 48.2)
- added K27: V23079C1103B301, SamacSys_Parts:V23079A1001B301, F.Cu at (166.4, 48.2)
- added K28: V23079C1103B301, SamacSys_Parts:V23079A1001B301, F.Cu at (194.3, 48.2)
- added K29: V23079C1103B301, SamacSys_Parts:V23079A1001B301, F.Cu at (137.2, 48.2)
- added K30: IMC03TS, SamacSys_Parts:IMC03TS, F.Cu at (153.9, 48.2)
- added K31: IMC03TS, SamacSys_Parts:IMC03TS, F.Cu at (180.6, 48.2)
- added K32: IMC03TS, SamacSys_Parts:IMC03TS, F.Cu at (123.2, 48.5)
- added K33: V23079C1103B301, SamacSys_Parts:V23079A1001B301, F.Cu at (279.9, 138.4)
- added K34: V23079C1103B301, SamacSys_Parts:V23079A1001B301, F.Cu at (279.9, 115.5)
- added K35: V23079C1103B301, SamacSys_Parts:V23079A1001B301, F.Cu at (279.9, 91.4)
- added K36: V23079C1103B301, SamacSys_Parts:V23079A1001B301, F.Cu at (279.9, 68.5)
- added K37: V23079C1103B301, SamacSys_Parts:V23079A1001B301, F.Cu at (256.0, 242.2)
- added K38: IMC03TS, SamacSys_Parts:IMC03TS, F.Cu at (279.9, 150.1)
- added K39: IMC03TS, SamacSys_Parts:IMC03TS, F.Cu at (279.9, 127.2)
- added K40: IMC03TS, SamacSys_Parts:IMC03TS, F.Cu at (279.9, 103.1)
- added K41: IMC03TS, SamacSys_Parts:IMC03TS, F.Cu at (279.6, 80.2)
- added K42: IMC03TS, SamacSys_Parts:IMC03TS, F.Cu at (255.8, 253.9)
- added K43: V23079C1103B301, SamacSys_Parts:V23079A1001B301, F.Cu at (256.0, 190.1)
- added K44: V23079C1103B301, SamacSys_Parts:V23079A1001B301, F.Cu at (254.8, 163.5)
- added K45: V23079C1103B301, SamacSys_Parts:V23079A1001B301, F.Cu at (256.0, 216.8)
- added K46: IMC03TS, SamacSys_Parts:IMC03TS, F.Cu at (254.8, 203.1)
- added K47: IMC03TS, SamacSys_Parts:IMC03TS, F.Cu at (254.1, 176.4)
- added K48: IMC03TS, SamacSys_Parts:IMC03TS, F.Cu at (256.0, 228.5)
- added Q1: 2N5457, SamacSys_Parts:PN4117, F.Cu at (84.0, 83.0)
- added Q2: 2N5457, SamacSys_Parts:PN4117, F.Cu at (73.0, 87.5)
- added U2: INA128, Package_SO:SOIC-8_3.9x4.9mm_P1.27mm, F.Cu at (59.0, 88.1)
- IC1, IC10, IC2, IC6, IC7, IC8: value DRDC3105F-7 -> TD62083AFGNEL; footprint Library:SOT96P240X110-3N -> SamacSys_Parts:SOIC127P1030X245-18N
- IC4, IC5: value DRDC3105F-7 -> MC74VHC138DR2G; footprint Library:SOT96P240X110-3N -> SamacSys_Parts:SOIC127P600X175-16N
- IC9: value DRDC3105F-7 -> LM358PWG4; footprint Library:SOT96P240X110-3N -> SamacSys_Parts:SOP65P640X120-8N
- J10: value DadConnector -> TENGConnector; footprint Connector_PinHeader_2.54mm:PinHeader_1x14_P2.54mm_Vertical -> SamacSys_Parts:231162001000
- J12: value Load 0 -> PH-2X05SG; footprint Connector_PinHeader_2.54mm:PinHeader_1x03_P2.54mm_Horizontal -> SamacSys_Parts:HDRV10W66P254_2X5_1270X500X895P
- K1, K11, K13, K15, K3, K5, K7, K9: footprint Library:V23079A1001B301 -> SamacSys_Parts:V23079A1001B301
- K10, K12, K14, K16, K2, K4, K6, K8: footprint Library:IMC03TS -> SamacSys_Parts:IMC03TS
- R1: value 0 -> R
- R5: footprint Resistor_THT:R_Axial_DIN0614_L14.3mm_D5.7mm_P20.32mm_Horizontal -> Resistor_SMD:R_0805_2012Metric
- moved J8 236.0 mm to (218.0, 265.1), turned to 90 degrees
- moved J3 208.0 mm to (84.7, 265.1), turned to -90 degrees
- moved K11 189.0 mm to (215.5, 238.5), turned to -90 degrees
- moved J6 188.9 mm to (163.4, 265.1), turned to 90 degrees
- moved K12 186.8 mm to (227.9, 237.8), turned to -90 degrees
- moved K6 178.4 mm to (73.2, 237.2), turned to -90 degrees
- moved J4 171.2 mm to (111.3, 265.1), turned to -90 degrees
- moved K5 170.9 mm to (87.2, 238.5), turned to -90 degrees
- moved IC2 166.7 mm to (184.5, 170.2), turned to 0 degrees
- moved K15 162.9 mm to (160.1, 237.9), turned to -90 degrees
- moved J7 158.3 mm to (191.3, 265.1), turned to 90 degrees
- moved J2 157.2 mm to (49.0, 211.0)
- moved R6 145.0 mm to (74.6, 81.0), turned to 180 degrees
- moved K16 142.1 mm to (173.3, 238.5), turned to -90 degrees
- moved J5 140.5 mm to (139.3, 265.1), turned to -90 degrees
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Connections:
- IC1 pad 2: GND -> /Y1
- IC1 pad 3: Net-(IC1-OUT) -> /Y2
- IC10 pad 1: /Y4 -> /Y16
- IC10 pad 2: GND -> /Y17
- IC10 pad 3: Net-(IC10-OUT) -> /Y18
- IC2 pad 2: GND -> /Y1
- IC2 pad 3: Net-(IC2-OUT) -> /Y2
- IC4 pad 1: /Y1 -> /Din0
- IC4 pad 2: GND -> /Din1
- IC4 pad 3: Net-(IC4-OUT) -> /Din2
- IC5 pad 1: /Y1 -> /Din0
- IC5 pad 2: GND -> /Din1
- IC5 pad 3: Net-(IC5-OUT) -> /Din2
- IC6 pad 1: /Y2 -> /Y8
- IC6 pad 2: GND -> /Y9
- IC6 pad 3: Net-(IC6-OUT) -> /Y10
- IC7 pad 1: /Y2 -> /Y8
- IC7 pad 2: GND -> /Y9
- IC7 pad 3: Net-(IC7-OUT) -> /Y10
- IC8 pad 1: /Y3 -> /Y16
- IC8 pad 2: GND -> /Y17
- IC8 pad 3: Net-(IC8-OUT) -> /Y18
- IC9 pad 1: /Y3 -> /Dout1
- IC9 pad 2: GND -> /Current_Sense1
- IC9 pad 3: Net-(IC9-OUT) -> GND
- J10 pad 1: /Din0 -> /Teng+
- J10 pad 2: /Din1 -> /TengN
- J12 pad 1: Net-(J12-Pin_1) -> /TengN
- J12 pad 2: Net-(J12-Pin_2) -> /TENG-
- J12 pad 3: Net-(J12-Pin_3) -> /Current_Sense1
- K1 pad 1: Net-(IC2-OUT) -> /O2
- K1 pad 4: /Loads/Rb_0 -> /Loads/Ra_0
- K1 pad 9: /Loads/Rc_0 -> /Loads/Rb_0
- K10 pad 1: Net-(IC10-OUT) -> /O9
- K11 pad 1: Net-(IC13-OUT) -> /O12
- K11 pad 4: /Loads/Rb_5 -> /Loads/Ra_5
- K11 pad 9: /Loads/Ra_5 -> /Loads/Rb_5
- K12 pad 1: Net-(IC12-OUT) -> /O11
- K13 pad 1: Net-(IC15-OUT) -> /O14
- K13 pad 4: /Loads/Rb_6 -> /Loads/Ra_6
- K13 pad 9: /Loads/Ra_6 -> /Loads/Rb_6
- K14 pad 1: Net-(IC14-OUT) -> /O13
- K15 pad 1: Net-(IC17-OUT) -> /O16
- K15 pad 4: /Loads/Rb_7 -> /Loads/Ra_7
- K15 pad 9: /Loads/Ra_7 -> /Loads/Rb_7
- K16 pad 1: Net-(IC16-OUT) -> /O15
- K2 pad 1: Net-(IC1-OUT) -> /O1
- K2 pad 3: /Loads/Ra_0 -> /Loads/Rc_0
- K3 pad 1: Net-(IC5-OUT) -> /O4
- K3 pad 4: /Loads/Rb_1 -> /Loads/Ra_1
- K3 pad 9: /Loads/Ra_1 -> /Loads/Rb_1
- K4 pad 1: Net-(IC4-OUT) -> /O3
- K5 pad 1: Net-(IC7-OUT) -> /O6
- K5 pad 4: /Loads/Rb_2 -> /Loads/Ra_2
- K5 pad 9: /Loads/Ra_2 -> /Loads/Rb_2
- K6 pad 1: Net-(IC6-OUT) -> /O5
- K7 pad 1: Net-(IC9-OUT) -> /O8
- K7 pad 4: /Loads/Rb_3 -> /Loads/Ra_3
- K7 pad 9: /Loads/Ra_3 -> /Loads/Rb_3
- K8 pad 1: Net-(IC8-OUT) -> /O7
- K9 pad 1: Net-(IC11-OUT) -> /O10
- K9 pad 4: /Loads/Rb_4 -> /Loads/Ra_4
- K9 pad 9: /Loads/Ra_4 -> /Loads/Rb_4
- R1 pad 1: Net-(J10-Pin_14) -> Net-(Q1-G)
- R2 pad 1: Net-(R2-Pad1) -> /Dout1
- R2 pad 2: Net-(J12-Pin_3) -> /Current_Sense1
- R3 pad 1: Net-(R3-Pad1) -> /Current_Sense2
- R3 pad 2: Net-(J12-Pin_3) -> Net-(JP2-A)
- R4 pad 1: Net-(J12-Pin_2) -> Net-(R4-Pad1)
- R4 pad 2: Net-(R3-Pad1) -> Net-(R4-Pad2)
- R5 pad 1: Net-(J12-Pin_1) -> Net-(Q2-S)
- R5 pad 2: Net-(R2-Pad1) -> GND
- R6 pad 2: Net-(J12-Pin_2) -> Net-(Q2-G)
Routing:
- net /Din2: track 31.7 -> 0.00 mm
- net /Din1: track 31.0 -> 0.00 mm
- net /Din0: track 30.5 -> 0.00 mm
- net /Loads/Ra_0: track 17.4 -> 0.00 mm
- net /Loads/Rb_0: track 16.1 -> 0.00 mm
- net /Loads/Rc_0: track 9.56 -> 0.00 mm
Other:
- board size 143.5 x 116.5 mm -> 357 x 270.5 mm

Commit message: new 08/11
Parts:
- removed C5, C6: 100nF, Capacitor_SMD:C_0805_2012Metric
- removed J1, J14, J23: Load 0, Connector_PinHeader_2.54mm:PinHeader_1x03_P2.54mm_Vertical
- removed J10: TENGConnector, SamacSys_Parts:231162001000
- removed J11: TENG, Connector_PinHeader_2.54mm:PinHeader_1x02_P2.54mm_Vertical
- removed J15, J2, J24: Load 1, Connector_PinHeader_2.54mm:PinHeader_1x03_P2.54mm_Vertical
- removed J16, J25, J3: Load 2, Connector_PinHeader_2.54mm:PinHeader_1x03_P2.54mm_Vertical
- removed J17, J26, J4: Load 3, Connector_PinHeader_2.54mm:PinHeader_1x03_P2.54mm_Vertical
- removed J18, J27, J5: Load 4, Connector_PinHeader_2.54mm:PinHeader_1x03_P2.54mm_Vertical
- removed J19: DaqConnector, SamacSys_Parts:231339001000
- removed J20, J29, J7: Load 6, Connector_PinHeader_2.54mm:PinHeader_1x03_P2.54mm_Vertical
- removed J21, J6: Load 7, Connector_PinHeader_2.54mm:PinHeader_1x03_P2.54mm_Vertical
- removed J22, J31, J8: Load 5, Connector_PinHeader_2.54mm:PinHeader_1x03_P2.54mm_Vertical
- removed Q1, Q2: 2N5457, SamacSys_Parts:PN4117
- removed R1, R5, R6: R, Resistor_SMD:R_0805_2012Metric
- added IC11: MC74VHC138DR2G, SamacSys_Parts:SOIC127P600X175-16N, F.Cu at (203.2, 188.7)
- added J13: 1757242, SamacSys_Parts:1757242, F.Cu at (73.0, 155.9)
- added Load_0: Load 0, Connector_PinHeader_2.54mm:PinHeader_1x03_P2.54mm_Vertical, F.Cu at (93.5, 62.5)
- added Load_1: Load 1, Connector_PinHeader_2.54mm:PinHeader_1x03_P2.54mm_Vertical, F.Cu at (130.5, 62.9)
- added Load_10: Load 10, Connector_PinHeader_2.54mm:PinHeader_1x03_P2.54mm_Vertical, F.Cu at (383.3, 162.7)
- added Load_11: Load 11, Connector_PinHeader_2.54mm:PinHeader_1x03_P2.54mm_Vertical, F.Cu at (383.8, 191.7)
- added Load_12: Load 12, Connector_PinHeader_2.54mm:PinHeader_1x03_P2.54mm_Vertical, F.Cu at (383.3, 220.2)
- added Load_13: Load 13, Connector_PinHeader_2.54mm:PinHeader_1x03_P2.54mm_Vertical, F.Cu at (383.3, 246.7)
- added Load_14: Load 14, Connector_PinHeader_2.54mm:PinHeader_1x03_P2.54mm_Vertical, F.Cu at (382.8, 274.7)
- added Load_15: Load 15, Connector_PinHeader_2.54mm:PinHeader_1x03_P2.54mm_Vertical, F.Cu at (376.8, 308.2)
- added Load_16: Load 16, Connector_PinHeader_2.54mm:PinHeader_1x03_P2.54mm_Vertical, F.Cu at (347.8, 351.8)
- added Load_17: Load 17, Connector_PinHeader_2.54mm:PinHeader_1x03_P2.54mm_Vertical, F.Cu at (316.8, 351.8)
- added Load_18: Load 18, Connector_PinHeader_2.54mm:PinHeader_1x03_P2.54mm_Vertical, F.Cu at (282.3, 350.8)
- added Load_19: Load 19, Connector_PinHeader_2.54mm:PinHeader_1x03_P2.54mm_Vertical, F.Cu at (246.3, 350.8)
- added Load_2: Load 2, Connector_PinHeader_2.54mm:PinHeader_1x03_P2.54mm_Vertical, F.Cu at (163.0, 63.9)
- added Load_20: Load 20, Connector_PinHeader_2.54mm:PinHeader_1x03_P2.54mm_Vertical, F.Cu at (206.3, 350.3)
- added Load_21: Load 21, Connector_PinHeader_2.54mm:PinHeader_1x03_P2.54mm_Vertical, F.Cu at (167.8, 344.7)
- added Load_22: Load 22, Connector_PinHeader_2.54mm:PinHeader_1x03_P2.54mm_Vertical, F.Cu at (129.8, 344.7)
- added Load_23: Load 23, Connector_PinHeader_2.54mm:PinHeader_1x03_P2.54mm_Vertical, F.Cu at (89.3, 344.7)
- added Load_3: Load 3, Connector_PinHeader_2.54mm:PinHeader_1x03_P2.54mm_Vertical, F.Cu at (197.5, 64.0)
- added Load_4: Load 4, Connector_PinHeader_2.54mm:PinHeader_1x03_P2.54mm_Vertical, F.Cu at (232.5, 64.0)
- added Load_5: Load 5, Connector_PinHeader_2.54mm:PinHeader_1x03_P2.54mm_Vertical, F.Cu at (266.0, 64.5)
- added Load_6: Load 6, Connector_PinHeader_2.54mm:PinHeader_1x03_P2.54mm_Vertical, F.Cu at (300.5, 65.0)
- added Load_7: Load 7, Connector_PinHeader_2.54mm:PinHeader_1x03_P2.54mm_Vertical, F.Cu at (336.5, 70.1)
- added Load_8: Load 8, Connector_PinHeader_2.54mm:PinHeader_1x03_P2.54mm_Vertical, F.Cu at (383.8, 102.2)
- added Load_9: Load 9, Connector_PinHeader_2.54mm:PinHeader_1x03_P2.54mm_Vertical, F.Cu at (382.8, 133.2)
- added TENG_Connector1: Conn_01x04_Pin, Connector_PinHeader_2.54mm:PinHeader_1x04_P2.54mm_Vertical, F.Cu at (74.5, 130.0)
- IC1: value TD62083AFGNEL -> OPA2145IDR; footprint SamacSys_Parts:SOIC127P1030X245-18N -> SamacSys_Parts:SOIC127P600X175-8N
- IC3: value MC74VHC138DR2G -> TD62083AFGNEL; footprint Library:SOIC127P600X175-16N -> SamacSys_Parts:SOIC127P1030X245-18N
- J30: value Load 7 -> 1757349; footprint Connector_PinHeader_2.54mm:PinHeader_1x03_P2.54mm_Vertical -> SamacSys_Parts:SHDRRA12W103P0X508_1X12_6296X1200X875P
- K12, K2, K4: value IMC03TS -> V23079C1103B301; footprint SamacSys_Parts:IMC03TS -> SamacSys_Parts:V23079A1001B301
- K15, K7, K9: value V23079C1103B301 -> IMC03TS; footprint SamacSys_Parts:V23079A1001B301 -> SamacSys_Parts:IMC03TS
- moved K26 288.0 mm to (314.0, 234.0), turned to 180 degrees
- moved K21 282.3 mm to (312.0, 243.3), turned to 0 degrees
- moved K32 280.1 mm to (314.3, 253.2), turned to 180 degrees
- moved K28 278.2 mm to (312.0, 300.3), turned to 0 degrees
- moved K31 277.4 mm to (314.3, 291.2), turned to 180 degrees
- moved K29 276.4 mm to (312.0, 262.3), turned to 0 degrees
- moved K30 275.2 mm to (314.0, 272.0), turned to 180 degrees
- moved K27 274.8 mm to (312.0, 281.3), turned to 0 degrees
- moved K36 244.7 mm to (206.1, 301.8), turned to -90 degrees
- moved J30 237.3 mm to (72.5, 246.0), turned to 90 degrees
- moved C2 234.7 mm to (90.2, 285.8)
- moved C1 232.9 mm to (109.0, 284.5), turned to -90 degrees
- moved K41 228.5 mm to (215.4, 299.5), turned to -90 degrees
- moved C3 221.8 mm to (132.0, 247.1), turned to -90 degrees
- moved K35 217.6 mm to (225.6, 302.2), turned to -90 degrees
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Connections:
- net /Current_Sense1 renamed /Current_Sense1_IN
- net /Current_Sense2 renamed /Current_Sense2_IN
- net /O17 renamed /2_Loads/O17
- net /O18 renamed /2_Loads/O18
- net /O19 renamed /2_Loads/O19
- net /O20 renamed /2_Loads/O20
- net /O21 renamed /2_Loads/O21
- net /O22 renamed /2_Loads/O22
- net /O23 renamed /2_Loads/O23
- net /O24 renamed /2_Loads/O24
- net /O25 renamed /2_Loads/O25
- net /O26 renamed /2_Loads/O26
- net /O27 renamed /2_Loads/O27
- net /O28 renamed /2_Loads/O28
- net /O29 renamed /2_Loads/O29
- net /O30 renamed /2_Loads/O30
- net /O31 renamed /2_Loads/O31
- net /O32 renamed /2_Loads/O32
- net /O33 renamed /3_Loads/O33
- net /O34 renamed /3_Loads/O34
- net /O35 renamed /3_Loads/O35
- net /O36 renamed /3_Loads/O36
- net /O37 renamed /3_Loads/O37
- net /O38 renamed /3_Loads/O38
- net /O39 renamed /3_Loads/O39
- net /O40 renamed /3_Loads/O40
- net /O41 renamed /3_Loads/O41
- net /O42 renamed /3_Loads/O42
- net /O43 renamed /3_Loads/O43
- net /O44 renamed /3_Loads/O44
- net /O45 renamed /3_Loads/O45
- net /O46 renamed /3_Loads/O46
- net /O47 renamed /3_Loads/O47
- net /O48 renamed /3_Loads/O48
- net /Y10 renamed /2_Loads/Y10
- net /Y11 renamed /2_Loads/Y11
- net /Y12 renamed /2_Loads/Y12
- net /Y13 renamed /2_Loads/Y13
- net /Y14 renamed /2_Loads/Y14
- net /Y15 renamed /2_Loads/Y15
- net /Y16 renamed /3_Loads/Y16
- net /Y17 renamed /3_Loads/Y17
- net /Y18 renamed /3_Loads/Y18
- net /Y19 renamed /3_Loads/Y19
- net /Y20 renamed /3_Loads/Y20
- net /Y21 renamed /3_Loads/Y21
- net /Y22 renamed /3_Loads/Y22
- net /Y23 renamed /3_Loads/Y23
- net /Y8 renamed /2_Loads/Y8
- net /Y9 renamed /2_Loads/Y9
- IC1 pad 1: /Y0 -> Net-(IC1-+IN_B)
- IC1 pad 2: /Y1 -> Net-(IC1-+IN_B)
- IC1 pad 3: /Y2 -> /Vsense
- IC1 pad 4: /Y3 -> GND
- IC1 pad 5: /Y4 -> Net-(IC1-+IN_B)
- IC1 pad 6: /Y5 -> /V_daq
- IC1 pad 7: /Y6 -> /V_daq
- IC1 pad 8: /Y7 -> VCC
- IC2 pad 1: /Y0 -> /1_Loads/Y0
- IC2 pad 11: /O16 -> /1_Loads/O8
- IC2 pad 12: /O15 -> /1_Loads/O7
- IC2 pad 13: /O14 -> /1_Loads/O6
- IC2 pad 14: /O13 -> /1_Loads/O5
- IC2 pad 15: /O12 -> /1_Loads/O4
- IC2 pad 16: /O11 -> /1_Loads/O3
- IC2 pad 17: /O10 -> /1_Loads/O2
- IC2 pad 18: /O9 -> /1_Loads/O1
- IC2 pad 2: /Y1 -> /1_Loads/Y1
- IC2 pad 3: /Y2 -> /1_Loads/Y2
- IC2 pad 4: /Y3 -> /1_Loads/Y3
- IC2 pad 5: /Y4 -> /1_Loads/Y4
- IC2 pad 6: /Y5 -> /1_Loads/Y5
- IC2 pad 7: /Y6 -> /1_Loads/Y6
- IC2 pad 8: /Y7 -> /1_Loads/Y7
- IC3 pad 1: /Din0 -> /1_Loads/Y0
- IC3 pad 10: /Y5 -> VCC
- IC3 pad 11: /Y4 -> /1_Loads/O16
- IC3 pad 12: /Y3 -> /1_Loads/O15
- IC3 pad 13: /Y2 -> /1_Loads/O14
- IC3 pad 14: /Y1 -> /1_Loads/O13
- IC3 pad 15: /Y0 -> /1_Loads/O12
- IC3 pad 16: VCC -> /1_Loads/O11
- IC3 pad 2: /Din1 -> /1_Loads/Y1
- IC3 pad 3: /Din2 -> /1_Loads/Y2
- IC3 pad 4: /Din3 -> /1_Loads/Y3
- IC3 pad 5: /Din4 -> /1_Loads/Y4
- IC3 pad 6: /Din5 -> /1_Loads/Y5
- IC3 pad 7: /Y7 -> /1_Loads/Y6
- IC3 pad 8: GND -> /1_Loads/Y7
- IC3 pad 9: /Y6 -> GND
- J12 pad 10: /TENG- -> GND
- J12 pad 2: /TENG- -> /Teng-
- J12 pad 4: /TENG- -> /Teng-
- J12 pad 6: /TENG- -> /Teng-
- J12 pad 7: unconnected-(J12-Pad7) -> /Current_Sense2_OUT
- J12 pad 8: /TENG- -> /TengN
- J12 pad 9: GND -> /Current_Sense2_OUT
- J30 pad 1: /Loads2/Ra_7 -> /Vsense
- J30 pad 2: /Loads2/Rb_7 -> /V_daq
- J30 pad 3: /Loads2/Rc_7 -> /Din5
- K1 pad 1: /O2 -> /1_Loads/O2
- K1 pad 4: /Loads/Ra_0 -> /1_Loads/Loads-1/Ra_0
- K1 pad 9: /Loads/Rb_0 -> /1_Loads/Loads-1/Rb_0
- K10 pad 1: /O9 -> /1_Loads/O9
- K10 pad 3: /Loads/Rc_4 -> /1_Loads/Loads-1/Rc_4
- K11 pad 1: /O12 -> /1_Loads/O14
- K11 pad 4: /Loads/Ra_5 -> /1_Loads/Loads-1/Ra_6
- K11 pad 9: /Loads/Rb_5 -> /1_Loads/Loads-1/Rb_6
- K12 pad 1: /O11 -> /1_Loads/O16
- K12 pad 3: /Loads/Rc_5 -> unconnected-(K12-NC_1-Pad3)
- K12 pad 5: /Teng- -> /Teng+
- K12 pad 8: GND -> /Vsense
- K13 pad 1: /O14 -> /1_Loads/O12
- K13 pad 4: /Loads/Ra_6 -> /1_Loads/Loads-1/Ra_5
- K13 pad 9: /Loads/Rb_6 -> /1_Loads/Loads-1/Rb_5
- K14 pad 1: /O13 -> /1_Loads/O13
- K14 pad 3: /Loads/Rc_6 -> /1_Loads/Loads-1/Rc_6
- K15 pad 1: /O16 -> /1_Loads/O15
- K15 pad 3: unconnected-(K15-NC_1-Pad3) -> /1_Loads/Loads-1/Rc_7
- K15 pad 5: /Teng+ -> /Teng-
- K15 pad 8: /Vsense -> GND
- K16 pad 1: /O15 -> /1_Loads/O11
- K16 pad 3: /Loads/Rc_7 -> /1_Loads/Loads-1/Rc_5
- K17 pad 4: /Loads1/Ra_0 -> /2_Loads/Loads-2/Ra_0
- K17 pad 9: /Loads1/Rb_0 -> /2_Loads/Loads-2/Rb_0
- K18 pad 4: /Loads1/Ra_1 -> /2_Loads/Loads-2/Ra_1
- K18 pad 9: /Loads1/Rb_1 -> /2_Loads/Loads-2/Rb_1
- K19 pad 4: /Loads1/Ra_2 -> /2_Loads/Loads-2/Ra_2
- K19 pad 9: /Loads1/Rb_2 -> /2_Loads/Loads-2/Rb_2
- K2 pad 1: /O1 -> /1_Loads/O4
- K2 pad 3: /Loads/Rc_0 -> unconnected-(K2-NC_1-Pad3)
- K2 pad 5: /Teng- -> /Teng+
- K2 pad 8: GND -> /Vsense
- K20 pad 4: /Loads1/Ra_3 -> /2_Loads/Loads-2/Ra_3
- K20 pad 9: /Loads1/Rb_3 -> /2_Loads/Loads-2/Rb_3
- K21 pad 4: /Loads1/Ra_4 -> /2_Loads/Loads-2/Ra_4
- K21 pad 9: /Loads1/Rb_4 -> /2_Loads/Loads-2/Rb_4
- K22 pad 3: /Loads1/Rc_0 -> /2_Loads/Loads-2/Rc_0
- K23 pad 3: /Loads1/Rc_1 -> /2_Loads/Loads-2/Rc_1
- K24 pad 3: /Loads1/Rc_2 -> /2_Loads/Loads-2/Rc_2
- K25 pad 3: /Loads1/Rc_3 -> /2_Loads/Loads-2/Rc_3
- K26 pad 3: /Loads1/Rc_4 -> /2_Loads/Loads-2/Rc_4
- K27 pad 4: /Loads1/Ra_6 -> /2_Loads/Loads-2/Ra_6
- K27 pad 9: /Loads1/Rb_6 -> /2_Loads/Loads-2/Rb_6
- K28 pad 4: /Loads1/Ra_7 -> /2_Loads/Loads-2/Ra_7
- K28 pad 9: /Loads1/Rb_7 -> /2_Loads/Loads-2/Rb_7
- K29 pad 4: /Loads1/Ra_5 -> /2_Loads/Loads-2/Ra_5
- K29 pad 9: /Loads1/Rb_5 -> /2_Loads/Loads-2/Rb_5
- K3 pad 1: /O4 -> /1_Loads/O6
- K3 pad 4: /Loads/Ra_1 -> /1_Loads/Loads-1/Ra_2
- K3 pad 9: /Loads/Rb_1 -> /1_Loads/Loads-1/Rb_2
- K30 pad 3: /Loads1/Rc_6 -> /2_Loads/Loads-2/Rc_6
- K31 pad 3: /Loads1/Rc_7 -> /2_Loads/Loads-2/Rc_7
- K32 pad 3: /Loads1/Rc_5 -> /2_Loads/Loads-2/Rc_5
- K33 pad 4: /Loads2/Ra_0 -> /3_Loads/Loads-3/Ra_0
- K33 pad 9: /Loads2/Rb_0 -> /3_Loads/Loads-3/Rb_0
- K34 pad 4: /Loads2/Ra_1 -> /3_Loads/Loads-3/Ra_1
- K34 pad 9: /Loads2/Rb_1 -> /3_Loads/Loads-3/Rb_1
- K35 pad 4: /Loads2/Ra_2 -> /3_Loads/Loads-3/Ra_2
- K35 pad 9: /Loads2/Rb_2 -> /3_Loads/Loads-3/Rb_2
- K36 pad 4: /Loads2/Ra_3 -> /3_Loads/Loads-3/Ra_3
- K36 pad 9: /Loads2/Rb_3 -> /3_Loads/Loads-3/Rb_3
- K37 pad 4: /Loads2/Ra_4 -> /3_Loads/Loads-3/Ra_4
- K37 pad 9: /Loads2/Rb_4 -> /3_Loads/Loads-3/Rb_4
- K38 pad 3: /Loads2/Rc_0 -> /3_Loads/Loads-3/Rc_0
- K39 pad 3: /Loads2/Rc_1 -> /3_Loads/Loads-3/Rc_1
- K4 pad 1: /O3 -> /1_Loads/O8
- K4 pad 3: /Loads/Rc_1 -> unconnected-(K4-NC_1-Pad3)
- K4 pad 5: /Teng- -> /Teng+
- K4 pad 8: GND -> /Vsense
- K40 pad 3: /Loads2/Rc_2 -> /3_Loads/Loads-3/Rc_2
- K41 pad 3: /Loads2/Rc_3 -> /3_Loads/Loads-3/Rc_3
- K42 pad 3: /Loads2/Rc_4 -> /3_Loads/Loads-3/Rc_4
- K43 pad 4: /Loads2/Ra_6 -> /3_Loads/Loads-3/Ra_6
- K43 pad 9: /Loads2/Rb_6 -> /3_Loads/Loads-3/Rb_6
- K44 pad 4: /Loads2/Ra_7 -> /3_Loads/Loads-3/Ra_7
- K44 pad 9: /Loads2/Rb_7 -> /3_Loads/Loads-3/Rb_7
- K45 pad 4: /Loads2/Ra_5 -> /3_Loads/Loads-3/Ra_5
- K45 pad 9: /Loads2/Rb_5 -> /3_Loads/Loads-3/Rb_5
- K46 pad 3: /Loads2/Rc_6 -> /3_Loads/Loads-3/Rc_6
- K47 pad 3: /Loads2/Rc_7 -> /3_Loads/Loads-3/Rc_7
- K48 pad 3: /Loads2/Rc_5 -> /3_Loads/Loads-3/Rc_5
- K5 pad 1: /O6 -> /1_Loads/O10
- K5 pad 4: /Loads/Ra_2 -> /1_Loads/Loads-1/Ra_4
- K5 pad 9: /Loads/Rb_2 -> /1_Loads/Loads-1/Rb_4
- K6 pad 1: /O5 -> /1_Loads/O1
- K6 pad 3: /Loads/Rc_2 -> /1_Loads/Loads-1/Rc_0
- K7 pad 1: /O8 -> /1_Loads/O3
- K7 pad 3: unconnected-(K7-NC_1-Pad3) -> /1_Loads/Loads-1/Rc_1
- K7 pad 5: /Teng+ -> /Teng-
- K7 pad 8: /Vsense -> GND
- K8 pad 1: /O7 -> /1_Loads/O5
- K8 pad 3: /Loads/Rc_3 -> /1_Loads/Loads-1/Rc_2
- K9 pad 1: /O10 -> /1_Loads/O7
- K9 pad 3: unconnected-(K9-NC_1-Pad3) -> /1_Loads/Loads-1/Rc_3
- K9 pad 5: /Teng+ -> /Teng-
- K9 pad 8: /Vsense -> GND
- R3 pad 2: Net-(JP2-A) -> /Current_Sense2_OUT
- U2 pad 2: Net-(JP2-A) -> /Current_Sense2_OUT
Other:
- board size 357 x 270.5 mm -> 353 x 316.5 mm

Commit message: new 08/11
Parts:
- removed IC9: LM358PWG4, SamacSys_Parts:SOP65P640X120-8N
- removed JP2: Jumper_3_Bridged12, Jumper:SolderJumper-3_P1.3mm_Bridged2Bar12_Pad1.0x1.5mm_NumberLabels
- removed R2: R, Resistor_SMD:R_0805_2012Metric
- added IC12: OPA387DBVR, SamacSys_Parts:SOT95P280X145-5N, F.Cu at (236.0, 164.4)
- added R1: R, Resistor_SMD:R_0805_2012Metric, F.Cu at (207.8, 180.0)
- moved C2 115.8 mm to (202.4, 257.3)
- moved J9 97.6 mm to (161.5, 251.3)
- moved R3 96.6 mm to (182.1, 168.4)
- moved R4 96.6 mm to (192.5, 159.8)
- moved U2 96.6 mm to (192.6, 168.5)
- moved J30 89.5 mm to (158.5, 221.1)
- moved J13 89.3 mm to (159.0, 132.0)
- moved C4 87.5 mm to (198.1, 180.0), turned to -90 degrees
- moved Load_23 87.4 mm to (168.9, 308.5)
- moved Load_0 87.3 mm to (173.5, 97.5)
- moved TENG_Connector1 86.0 mm to (157.5, 107.4)
- moved C1 84.2 mm to (188.0, 255.3)
- moved U1 80.4 mm to (171.9, 250.1)
- moved Load_1 75.4 mm to (197.6, 97.5)
- moved C3 73.4 mm to (205.0, 239.4)
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Routing:
- net GND: track 0.00 -> 1095.3 mm, vias 0 -> 3
- net /Teng+: track 0.00 -> 647.0 mm, vias 0 -> 3
- net /Vsense: track 0.00 -> 644.0 mm, vias 0 -> 2
- net /Teng-: track 0.00 -> 544.3 mm, vias 0 -> 2
- net VCC: track 0.00 -> 496.1 mm, vias 0 -> 7
- net /Din1: track 0.00 -> 201.1 mm, vias 0 -> 1
- net /Din2: track 0.00 -> 198.5 mm, vias 0 -> 2
- net /Din4: track 0.00 -> 183.8 mm, vias 0 -> 2
- net /Din3: track 0.00 -> 183.7 mm, vias 0 -> 1
- net /Din0: track 0.00 -> 174.0 mm, vias 0 -> 1
- net /Din5: track 0.00 -> 168.1 mm, vias 0 -> 3
- net /TengN: track 0.00 -> 122.5 mm
- net /1_Loads/O1: track 0.00 -> 87.0 mm, vias 0 -> 1
- net /Dout1: track 0.00 -> 86.1 mm, vias 0 -> 1
- net /3_Loads/Y16: track 0.00 -> 85.9 mm, vias 0 -> 2
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Other:
- board size 353 x 316.5 mm -> 214.2 x 228.2 mm

Commit message: ruoting strategy
Parts:
- added C5: 100nF, Capacitor_SMD:C_0805_2012Metric, F.Cu at (181.6, 152.6)
- added C6: 100nF, Capacitor_SMD:C_0805_2012Metric, F.Cu at (278.5, 157.4)
- added C7: 100nF, Capacitor_SMD:C_0805_2012Metric, F.Cu at (261.1, 157.1)
- added C8: 100nF, Capacitor_SMD:C_0805_2012Metric, F.Cu at (346.3, 233.3)
- added C9: 100nF, Capacitor_SMD:C_0805_2012Metric, F.Cu at (251.6, 182.9)
- moved IC4 110.8 mm to (358.1, 261.3), turned to 0 degrees
- moved Load_8 91.6 mm to (433.6, 168.2)
- moved Load_9 86.5 mm to (433.6, 183.4)
- moved K17 81.8 mm to (403.9, 168.6)
- moved K18 81.8 mm to (403.9, 187.7)
- moved K19 81.8 mm to (403.9, 206.7)
- moved K20 81.8 mm to (404.4, 225.7)
- moved K21 81.8 mm to (404.4, 244.7)
- moved K22 81.8 mm to (405.9, 159.5)
- moved K23 81.8 mm to (406.2, 178.7)
- moved K24 81.8 mm to (406.3, 197.5)
- moved K25 81.8 mm to (406.2, 216.7)
- moved K26 81.8 mm to (406.4, 235.5)
- moved K27 81.8 mm to (404.4, 282.7)
- moved K28 81.8 mm to (404.4, 301.7)
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Routing:
- net GND: track 1095.3 -> 0.00 mm, vias 3 -> 0
- net /Teng+: track 647.0 -> 0.00 mm, vias 3 -> 0
- net /Vsense: track 644.0 -> 0.00 mm, vias 2 -> 0
- net /Teng-: track 544.3 -> 6.98 mm, vias 2 -> 0
- net VCC: track 496.1 -> 0.00 mm, vias 7 -> 0
- net /Din2: track 198.5 -> 0.00 mm, vias 2 -> 0
- net /Din4: track 183.8 -> 0.00 mm, vias 2 -> 0
- net /Din3: track 183.7 -> 0.00 mm, vias 1 -> 0
- net /Din0: track 174.0 -> 0.00 mm, vias 1 -> 0
- net /Din5: track 168.1 -> 0.00 mm, vias 3 -> 0
- net /TengN: track 122.5 -> 0.00 mm
- net /Din1: track 201.1 -> 100.8 mm, vias 1 -> 0
- net /Dout1: track 86.1 -> 0.00 mm, vias 1 -> 0
- net /3_Loads/Y16: track 85.9 -> 0.00 mm, vias 2 -> 0
- net /3_Loads/Y17: track 82.9 -> 0.00 mm, vias 2 -> 0
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