File: Project/load_automatisation.kicad_pcb (KiCad board)
At the start: 2 copper layers, 263.4 x 251.4 mm, 111 parts, among them IC1 OPA2145IDR, IC10 TD62083AFGNEL, IC11 MC74VHC138DR2G, IC12 OPA387DBVR, IC2 TD62083AFGNEL, IC3 TD62083AFGNEL, IC4 MC74VHC138DR2G, IC5 MC74VHC138DR2G, IC6 TD62083AFGNEL, IC7 TD62083AFGNEL, IC8 TD62083AFGNEL, J12 PH-2X05SG, J13 1757242, J30 1757349, J9 PowerIn, K1 V23079C1103B301, K10 IMC03TS, K11 V23079C1103B301, K12 V23079C1103B301, K13 V23079C1103B301, K14 IMC03TS, K15 IMC03TS, K16 IMC03TS, K17 V23079C1103B301, K18 V23079C1103B301, K19 V23079C1103B301, K2 V23079C1103B301, K20 V23079C1103B301, K21 V23079C1103B301, K22 IMC03TS, K23 IMC03TS, K24 IMC03TS, K25 IMC03TS, K26 IMC03TS, K27 V23079C1103B301, K28 V23079C1103B301, K29 V23079C1103B301, K3 V23079C1103B301, K30 IMC03TS, K31 IMC03TS, K32 IMC03TS, K33 V23079C1103B301, K34 V23079C1103B301, K35 V23079C1103B301, K36 V23079C1103B301, K37 V23079C1103B301, K38 IMC03TS, K39 IMC03TS, K4 V23079C1103B301, K40 IMC03TS, K41 IMC03TS, K42 IMC03TS, K43 V23079C1103B301, K44 V23079C1103B301, K45 V23079C1103B301, K46 IMC03TS, K47 IMC03TS, K48 IMC03TS, K5 V23079C1103B301, K6 IMC03TS, K7 IMC03TS, K8 IMC03TS, K9 IMC03TS, U1 AMS1117-5.0, U2 INA128

Commit message: routing 28/11
Routing:
- net /Teng-: track 786.6 -> 880.4 mm
- net /Vsense: track 854.5 -> 895.1 mm
- net /Teng+: track 936.5 -> 919.5 mm, vias 64 -> 22
- net VCC: track 879.4 -> 882.5 mm

Commit message: routing 28/11
Routing:
- net GND: track 1538.6 -> 1550.8 mm
- net /Teng+: track 919.5 -> 926.1 mm
- net /Teng-: track 880.4 -> 883.7 mm

Commit message: routing 03/12
Parts:
- removed IC12: OPA387DBVR, SamacSys_Parts:SOT95P280X145-5N
- added C15: 100uF, Capacitor_THT:CP_Radial_D8.0mm_P3.80mm, F.Cu at (138.4, 158.0)
- added C16: 100uF, Capacitor_THT:CP_Radial_D8.0mm_P3.80mm, F.Cu at (150.9, 148.1)
- added IC9: OPA145IDBVT, SamacSys_Parts:SOT95P280X145-5N, F.Cu at (208.3, 157.4)
- added J1: PowerNeg, Connector_PinHeader_2.54mm:PinHeader_1x02_P2.54mm_Vertical, F.Cu at (125.2, 158.0)
- added U3: AMS1117-5.0, Package_TO_SOT_SMD:SOT-223-3_TabPin2, F.Cu at (151.3, 156.2)
- moved C10 20.8 mm to (307.7, 241.6)
- moved C1 6.96 mm to (150.1, 174.0), turned to 90 degrees
- moved J9 5.13 mm to (124.7, 172.2)
- moved C11 2.98 mm to (254.8, 279.0)
Connections:
- IC1 pad 4: GND -> -VCC
- U2 pad 4: GND -> -VCC
Routing:
- net GND: track 1550.8 -> 1682.3 mm, vias 10 -> 9
- net -VCC: track 0.00 -> 62.4 mm, vias 0 -> 2
- net VCC: track 882.5 -> 915.6 mm
- net /VNeg: track 0.00 -> 23.1 mm
- net /Vin: track 46.6 -> 45.3 mm

Commit message: routing 10/12
Parts:
- moved C11 29.1 mm to (225.8, 281.4)
- moved C13 18.6 mm to (283.3, 233.4), turned to 180 degrees
- moved C12 17.9 mm to (208.1, 281.9)
- moved C14 16.6 mm to (233.9, 253.7), turned to 90 degrees
- moved C9 5.94 mm to (252.0, 180.9), turned to 180 degrees
- moved C8 3.82 mm to (310.2, 258.8)
- moved C15 3.82 mm to (138.7, 154.2), turned to -90 degrees
- moved C16 3.81 mm to (150.9, 144.3), turned to -90 degrees
- moved C6 0.96 mm to (278.6, 156.4)
- moved IC9 0.13 mm to (208.4, 157.5)
Connections:
- C15 pad 1: /VNeg -> GND
- C15 pad 2: GND -> /VNeg
- C16 pad 1: -VCC -> GND
- C16 pad 2: GND -> -VCC
Routing:
- net VCC: track 915.6 -> 666.4 mm, vias 7 -> 8
- net -VCC: track 62.4 -> 151.9 mm, vias 2 -> 8
- net GND: track 1682.3 -> 1617.8 mm, vias 9 -> 20
- net /Din5: track 241.5 -> 229.1 mm, vias 0 -> 2
- net /Current_Sense1_IN: track 54.5 -> 66.0 mm
- net /Din4: track 239.7 -> 229.6 mm, vias 5 -> 3
- net /Din3: track 239.1 -> 229.9 mm, vias 5 -> 3
- net /Din2: track 238.7 -> 230.0 mm, vias 5 -> 3
- net /Din1: track 237.7 -> 229.8 mm, vias 5 -> 3
- net /Din0: track 230.6 -> 233.6 mm, vias 4 -> 3
- added copper zone on B.Cu, net GND
- added copper zone on F.Cu, net VCC
