File: Project/load_automatisation.kicad_sch (KiCad schematic)
At the start: 34 parts, among them IC1 OPA2145IDR, IC12 OPA387DBVR, J1 PowerNeg, J12 PH-2X05SG, J13 1757242, J30 1757349, J9 PowerIn, U1 AMS1117-5.0, U2 INA128, U3 AMS1117-5.0

Commit message: abre alimentacio
Connections:
- net -VCC: now also C16.2; no longer C16.1
- net GND: now also C15.1, C16.1; no longer C15.2, C16.2
- net VNeg: now also C15.2; no longer C15.1
Other:
- moved on the sheet: C15, C16
