File: Project/load_automatisation.kicad_sch (KiCad schematic)
At the start: 34 parts, among them IC1 OPA2145IDR, IC12 OPA387DBVR, J1 PowerNeg, J12 PH-2X05SG, J13 1757242, J30 1757349, J9 PowerIn, U1 AMS1117-5.0, U2 INA128, U3 AMS1117-5.0

Commit message: routing 10/12
Parts:
- removed IC12: OPA387DBVR, SOT95P280X145-5N, symbol SamacSys_Parts:OPA387DBVR
- added IC9: OPA145IDBVT, SOT95P280X145-5N, symbol SamacSys_Parts:OPA145IDBVT
Connections:
- net -VCC: now also C16.2, IC1.4 (V-), U2.4 (V-), IC9.2 (V-); no longer C16.1
- net Current_Sense1_IN: now also IC9.4 (-IN)
- net Dout1: now also IC9.1 (OUT)
- net GND: now also C15.1, C16.1, IC9.3 (+IN); no longer C15.2, C16.2, IC1.4 (V-), U2.4 (V-)
- net VCC: now also IC9.5 (V+)
- net VNeg: now also C15.2; no longer C15.1
Other:
- moved on the sheet: C15, C16
Changed lines of the file:
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@@
 	(wire
 		(pts
-			(xy 35.56 60.96) (xy 35.56 68.58)
-		)
-		(stroke
-			(width 0)
-			(type default)
-		)
-	)
-	(wire
-		(pts
 			(xy 226.06 81.28) (xy 226.06 78.74)
 		)
@@
 	(wire
 		(pts
+			(xy 35.56 60.96) (xy 35.56 68.58)
+		)
+		(stroke
+			(width 0)
+			(type default)
+		)
+	)
+	(wire
+		(pts
 			(xy 90.17 99.06) (xy 93.98 99.06)
 		)
@@
 	(symbol
 		(lib_id "Device:C_Polarized")
-		(at 39.37 63.5 0)
+		(at 39.37 63.5 180)
 		(unit 1)
 		(exclude_from_sim no)
@@
 		(fields_autoplaced yes)
 		(property "Reference" "C15"
-			(at 43.18 61.3409 0)
+			(at 43.18 63.1189 0)
 			(effects
 				(font
 					(size 1.27 1.27)
 				)
-				(justify left)
+				(justify right)
 			)
 		)
 		(property "Value" "100uF"
-			(at 43.18 63.8809 0)
+			(at 43.18 65.6589 0)
 			(effects
 				(font
 					(size 1.27 1.27)
 				)
-				(justify left)
+				(justify right)
 			)
 		)
 		(property "Footprint" "Capacitor_THT:CP_Radial_D8.0mm_P3.80mm"
-			(at 40.3352 67.31 0)
+			(at 38.4048 59.69 0)
 			(effects
 				(font
@@
 	(symbol
 		(lib_id "Device:C_Polarized")
-		(at 71.12 62.23 0)
+		(at 71.12 62.23 180)
 		(unit 1)
 		(exclude_from_sim no)
@@
 		(fields_autoplaced yes)
 		(property "Reference" "C16"
-			(at 74.93 60.0709 0)
+			(at 74.93 61.8489 0)
 			(effects
 				(font
 					(size 1.27 1.27)
 				)
-				(justify left)
+				(justify right)
 			)
 		)
 		(property "Value" "100uF"
-			(at 74.93 62.6109 0)
+			(at 74.93 64.3889 0)
 			(effects
 				(font
 					(size 1.27 1.27)
 				)
-				(justify left)
+				(justify right)
 			)
 		)
 		(property "Footprint" "Capacitor_THT:CP_Radial_D8.0mm_P3.80mm"
-			(at 72.0852 66.04 0)
+			(at 70.1548 58.42 0)
 			(effects
 				(font
@@
 	)
 	(symbol
-		(lib_id "SamacSys_Parts:OPA387DBVR")
-		(at 191.77 81.28 0)
+		(lib_id "power:VCC")
+		(at 124.46 91.44 270)
 		(unit 1)
 		(exclude_from_sim no)
@@
 		(on_board yes)
 		(dnp no)
-		(fields_autoplaced yes)
-		(property "Reference" "IC12"
-			(at 204.47 73.66 0)
+		(property "Reference" "#PWR083"
+			(at 120.65 91.44 0)
 			(effects
 				(font
 					(size 1.27 1.27)
 				)
+				(hide yes)
 			)
 		)
-		(property "Value" "OPA387DBVR"
-			(at 204.47 76.2 0)
+		(property "Value" "VCC"
+			(at 128.27 91.4399 90)
 			(effects
 				(font
 					(size 1.27 1.27)
 				)
+				(justify left)
 			)
 		)
-		(property "Footprint" "SOT95P280X145-5N"
-			(at 213.36 176.2 0)
+		(property "Footprint" ""
+			(at 124.46 91.44 0)
 			(effects
 				(font
 					(size 1.27 1.27)
 				)
-				(justify left top)
 				(hide yes)
 			)
 		)
-		(property "Datasheet" "https://www.ti.com/lit/ds/symlink/opa387.pdf?ts=1635153405851&ref_url=https%253A%252F%252Fwww.ti.com%252F"
-			(at 213.36 276.2 0)
+		(property "Datasheet" ""
+			(at 124.46 91.44 0)
 			(effects
 				(font
 					(size 1.27 1.27)
 				)
-				(justify left top)
 				(hide yes)
 			)
 		)
-		(property "Description" "Precision Amplifiers Ultra-high precision (2 uV), zero-drift (0.003 uV/C), low-input-bias-current op amp (single)"
-			(at 191.77 81.28 0)
+		(property "Description" "Power symbol creates a global label with name \"VCC\""
+			(at 124.46 91.44 0)
 			(effects
 				(font
@@
 			)
 		)
-		(property "Height" "1.45"
-			(at 213.36 476.2 0)
+		(pin "1"
+		)
+		(instances
+			(project "load_automatisation"
+				(path "/e193aeee-7d8e-4a61-b3f1-51249c7839f9"
+					(reference "#PWR083")
+					(unit 1)
+				)
+			)
+		)
+	)
+	(symbol
+		(lib_id "power:GND")
+		(at 191.77 88.9 0)
+		(unit 1)
+		(exclude_from_sim no)
+		(in_bom yes)
+		(on_board yes)
+		(dnp no)
+		(fields_autoplaced yes)
+		(property "Reference" "#PWR037"
+			(at 191.77 95.25 0)
 			(effects
 				(font
 					(size 1.27 1.27)
 				)
-				(justify left top)
 				(hide yes)
 			)
 		)
-		(property "Manufacturer_Name" "Texas Instruments"
-			(at 213.36 576.2 0)
+		(property "Value" "GND"
+			(at 191.77 93.98 0)
 			(effects
 				(font
 					(size 1.27 1.27)
 				)
-				(justify left top)
-				(hide yes)
 			)
 		)
-		(property "Manufacturer_Part_Number" "OPA387DBVR"
-			(at 213.36 676.2 0)
+		(property "Footprint" ""
+			(at 191.77 88.9 0)
 			(effects
 				(font
 					(size 1.27 1.27)
 				)
-				(justify left top)
 				(hide yes)
 			)
 		)
-		(property "Arrow Part Number" "OPA387DBVR"
-			(at 213.36 776.2 0)
+		(property "Datasheet" ""
+			(at 191.77 88.9 0)
 			(effects
 				(font
 					(size 1.27 1.27)
 				)
-				(justify left top)
 				(hide yes)
 			)
 		)
-		(property "Arrow Price/Stock" "null?region=nac"
-			(at 213.36 876.2 0)
+		(property "Description" "Power symbol creates a global label with name \"GND\" , ground"
+			(at 191.77 88.9 0)
 			(effects
 				(font
 					(size 1.27 1.27)
 				)
-				(justify left top)
 				(hide yes)
 			)
 		)
-		(pin "2"
-		)
-		(pin "5"
-		)
-		(pin "3"
-		)
-		(pin "4"
-		)
 		(pin "1"
 		)
 		(instances
-			(project ""
+			(project "load_automatisation"
 				(path "/e193aeee-7d8e-4a61-b3f1-51249c7839f9"
-					(reference "IC12")
+					(reference "#PWR037")
 					(unit 1)
 				)
@@
 	)
 	(symbol
-		(lib_id "power:VCC")
-		(at 124.46 91.44 270)
+		(lib_id "SamacSys_Parts:OPA145IDBVT")
+		(at 191.77 81.28 0)
 		(unit 1)
 		(exclude_from_sim no)
@@
 		(on_board yes)
 		(dnp no)
-		(property "Reference" "#PWR083"
-			(at 120.65 91.44 0)
+		(fields_autoplaced yes)
+		(property "Reference" "IC9"
+			(at 204.47 73.66 0)
 			(effects
 				(font
 					(size 1.27 1.27)
 				)
-				(hide yes)
 			)
 		)
-		(property "Value" "VCC"
-			(at 128.27 91.4399 90)
+		(property "Value" "OPA145IDBVT"
+			(at 204.47 76.2 0)
 			(effects
 				(font
 					(size 1.27 1.27)
 				)
-				(justify left)
 			)
 		)
-		(property "Footprint" ""
-			(at 124.46 91.44 0)
+		(property "Footprint" "SOT95P280X145-5N"
+			(at 213.36 176.2 0)
 			(effects
 				(font
 					(size 1.27 1.27)
 				)
+				(justify left top)
 				(hide yes)
 			)
 		)
-		(property "Datasheet" ""
-			(at 124.46 91.44 0)
+		(property "Datasheet" "https://www.ti.com/lit/gpn/OPA145"
+			(at 213.36 276.2 0)
 			(effects
 				(font
 					(size 1.27 1.27)
 				)
+				(justify left top)
 				(hide yes)
 			)
 		)
-		(property "Description" "Power symbol creates a global label with name \"VCC\""
-			(at 124.46 91.44 0)
+		(property "Description" "Op Amp Single Low Noise Amplifier R-R O/P +/-18V/36V 5-Pin SOT-23 T/R"
+			(at 191.77 81.28 0)
 			(effects
 				(font
@@
 			)
 		)
-		(pin "1"
+		(property "Height" "1.45"
+			(at 213.36 476.2 0)
+			(effects
+				(font
+					(size 1.27 1.27)
+				)
+				(justify left top)
+				(hide yes)
+			)
 		)
-		(instances
-			(project "load_automatisation"
-				(path "/e193aeee-7d8e-4a61-b3f1-51249c7839f9"
-					(reference "#PWR083")
-					(unit 1)
+		(property "Manufacturer_Name" "Texas Instruments"
+			(at 213.36 576.2 0)
+			(effects
+				(font
+					(size 1.27 1.27)
 				)
+				(justify left top)
+				(hide yes)
 			)
 		)
-	)
-	(symbol
-		(lib_id "power:GND")
-		(at 191.77 88.9 0)
-		(unit 1)
-		(exclude_from_sim no)
-		(in_bom yes)
-		(on_board yes)
-		(dnp no)
-		(fields_autoplaced yes)
-		(property "Reference" "#PWR037"
-			(at 191.77 95.25 0)
+		(property "Manufacturer_Part_Number" "OPA145IDBVT"
+			(at 213.36 676.2 0)
 			(effects
 				(font
 					(size 1.27 1.27)
 				)
+				(justify left top)
 				(hide yes)
 			)
 		)
-		(property "Value" "GND"
-			(at 191.77 93.98 0)
+		(property "Mouser Part Number" "595-OPA145IDBVT"
+			(at 213.36 776.2 0)
 			(effects
 				(font
 					(size 1.27 1.27)
 				)
+				(justify left top)
+				(hide yes)
 			)
 		)
-		(property "Footprint" ""
-			(at 191.77 88.9 0)
+		(property "Mouser Price/Stock" "https://www.mouser.co.uk/ProductDetail/Texas-Instruments/OPA145IDBVT?qs=w%2Fv1CP2dgqoYEgtccAiQSA%3D%3D"
+			(at 213.36 876.2 0)
 			(effects
 				(font
 					(size 1.27 1.27)
 				)
+				(justify left top)
 				(hide yes)
 			)
 		)
-		(property "Datasheet" ""
-			(at 191.77 88.9 0)
+		(property "Arrow Part Number" "OPA145IDBVT"
+			(at 213.36 976.2 0)
 			(effects
 				(font
 					(size 1.27 1.27)
 				)
+				(justify left top)
 				(hide yes)
 			)
 		)
-		(property "Description" "Power symbol creates a global label with name \"GND\" , ground"
-			(at 191.77 88.9 0)
+		(property "Arrow Price/Stock" "https://www.arrow.com/en/products/opa145idbvt/texas-instruments?region=nac"
+			(at 213.36 1076.2 0)
 			(effects
 				(font
 					(size 1.27 1.27)
 				)
+				(justify left top)
 				(hide yes)
 			)
 		)
+		(pin "2"
+		)
 		(pin "1"
 		)
+		(pin "3"
+		)
+		(pin "4"
+		)
+		(pin "5"
+		)
 		(instances
-			(project "load_automatisation"
+			(project ""
 				(path "/e193aeee-7d8e-4a61-b3f1-51249c7839f9"
-					(reference "#PWR037")
+					(reference "IC9")
 					(unit 1)
 				)
@@
 			)
 		)
-		(property "Value" "GND"
+		(property "Value" "-VCC"
 			(at 247.396 127.508 0)
 			(effects
@@
 			)
 		)
-		(property "Value" "GND"
+		(property "Value" "-VCC"
 			(at 89.916 103.378 0)
 			(effects
