File: Project/load_automatisation.kicad_sch (KiCad schematic)
At the start: 34 parts, among them IC1 OPA2145IDR, IC9 OPA145IDBVT, J1 PowerNeg, J12 PH-2X05SG, J13 1757242, J30 1757349, J9 PowerIn, U1 AMS1117-5.0, U2 INA128, U3 AMS1117-5.0

Commit message: place arrangement
Parts:
- removed C6, C7, C9: 100nF, Capacitor_SMD:C_0805_2012Metric, symbol Device:C
- added C17, C18: 100nF, Capacitor_SMD:C_0805_2012Metric, symbol Device:C
Connections:
- net -VCC: now also C17.1, C18.1
- net GND: now also C17.2, C18.2
- net V_daq+: now also J30.2; no longer J30.10
- net V_daq-: now also J30.1; no longer J30.9
Other:
- moved on the sheet: J30

Commit message: routing 11/12
Parts:
- removed C10, C11, C12, C13, C14, C8: 100nF, Capacitor_SMD:C_0805_2012Metric, symbol Device:C
- added C19, C20: 100nF, Capacitor_SMD:C_0805_2012Metric, symbol Device:C
Connections:
- net -VCC: now also C19.1
- net Dout1: now also J30.11; no longer J30.12
- net Dout2: now also J30.12; no longer J30.11
- net GND: now also C19.2, C20.2
- net VCC: now also C20.1
- net V_daq+: now also J30.1; no longer J30.2
- net V_daq-: now also J30.2; no longer J30.1

Commit message: new routing 12/12
Parts:
- IC1: footprint SOIC127P600X175-8N -> SamacSys_Parts:SOIC127P600X175-8N
- IC9: footprint SOT95P280X145-5N -> SamacSys_Parts:SOT95P280X145-5N
- J12: footprint HDRV10W66P254_2X5_1270X500X895P -> SamacSys_Parts:HDRV10W66P254_2X5_1270X500X895P
- J13: footprint 1757242 -> SamacSys_Parts:1757242
- J30: footprint SHDRRA12W103P0X508_1X12_6296X1200X875P -> SamacSys_Parts:SHDRRA12W103P0X508_1X12_6296X1200X875P
Changed lines of the file:
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@@
 			)
 		)
-		(property "Footprint" "HDRV10W66P254_2X5_1270X500X895P"
+		(property "Footprint" "SamacSys_Parts:HDRV10W66P254_2X5_1270X500X895P"
 			(at 162.56 225.73 0)
 			(effects
@@
 			)
 		)
-		(property "Footprint" "SHDRRA12W103P0X508_1X12_6296X1200X875P"
+		(property "Footprint" "SamacSys_Parts:SHDRRA12W103P0X508_1X12_6296X1200X875P"
 			(at 67.31 182.55 0)
 			(effects
@@
 			)
 		)
-		(property "Footprint" "SOT95P280X145-5N"
+		(property "Footprint" "SamacSys_Parts:SOT95P280X145-5N"
 			(at 213.36 176.2 0)
 			(effects
@@
 			)
 		)
-		(property "Footprint" "1757242"
+		(property "Footprint" "SamacSys_Parts:1757242"
 			(at 57.15 224.46 0)
 			(effects
@@
 			)
 		)
-		(property "Footprint" "SOIC127P600X175-8N"
+		(property "Footprint" "SamacSys_Parts:SOIC127P600X175-8N"
 			(at 120.65 186.36 0)
 			(effects
