File: Project/load_automatisation.kicad_sch (KiCad schematic)
At the start: 29 parts, among them IC1 OPA2145IDR, IC9 OPA145IDBVT, J1 PowerNeg, J12 PH-2X05SG, J13 1757242, J30 1757349, J9 PowerIn, U1 AMS1117-5.0, U2 INA128, U3 AMS1117-5.0

Commit message: new 16/01
Parts:
- added TENG_Connector2: Conn_01x04_Pin, Connector_PinHeader_2.54mm:PinHeader_1x04_P2.54mm_Vertical, symbol Connector:Conn_01x04_Pin
Connections:
- no-connect marks 0 -> 4
Changed lines of the file:
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@@
 		(color 0 0 0 0)
 	)
+	(no_connect
+		(at 45.72 171.45)
+	)
+	(no_connect
+		(at 45.72 163.83)
+	)
+	(no_connect
+		(at 45.72 166.37)
+	)
+	(no_connect
+		(at 45.72 168.91)
+	)
 	(wire
 		(pts
@@
 	(wire
 		(pts
+			(xy 45.72 163.83) (xy 40.64 163.83)
+		)
+		(stroke
+			(width 0)
+			(type default)
+		)
+	)
+	(wire
+		(pts
 			(xy 242.57 73.66) (xy 242.57 76.2)
 		)
@@
 	(wire
 		(pts
+			(xy 45.72 166.37) (xy 40.64 166.37)
+		)
+		(stroke
+			(width 0)
+			(type default)
+		)
+	)
+	(wire
+		(pts
 			(xy 135.89 130.81) (xy 143.51 130.81)
 		)
@@
 	(wire
 		(pts
+			(xy 45.72 168.91) (xy 40.64 168.91)
+		)
+		(stroke
+			(width 0)
+			(type default)
+		)
+	)
+	(wire
+		(pts
 			(xy 217.17 81.28) (xy 226.06 81.28)
 		)
@@
 	(wire
 		(pts
+			(xy 45.72 171.45) (xy 40.64 171.45)
+		)
+		(stroke
+			(width 0)
+			(type default)
+		)
+	)
+	(wire
+		(pts
 			(xy 90.17 99.06) (xy 93.98 99.06)
 		)
@@
 					(unit 1)
 				)
+			)
+		)
+	)
+	(symbol
+		(lib_id "Connector:Conn_01x04_Pin")
+		(at 35.56 166.37 0)
+		(unit 1)
+		(exclude_from_sim no)
+		(in_bom yes)
+		(on_board yes)
+		(dnp no)
+		(fields_autoplaced yes)
+		(property "Reference" "TENG_Connector2"
+			(at 36.195 158.75 0)
+			(effects
+				(font
+					(size 1.27 1.27)
+				)
+			)
+		)
+		(property "Value" "Conn_01x04_Pin"
+			(at 36.195 161.29 0)
+			(effects
+				(font
+					(size 1.27 1.27)
+				)
+			)
+		)
+		(property "Footprint" "Connector_PinHeader_2.54mm:PinHeader_1x04_P2.54mm_Vertical"
+			(at 35.56 166.37 0)
+			(effects
+				(font
+					(size 1.27 1.27)
+				)
+				(hide yes)
+			)
+		)
+		(property "Datasheet" "~"
+			(at 35.56 166.37 0)
+			(effects
+				(font
+					(size 1.27 1.27)
+				)
+				(hide yes)
+			)
+		)
+		(property "Description" "Generic connector, single row, 01x04, script generated"
+			(at 35.56 166.37 0)
+			(effects
+				(font
+					(size 1.27 1.27)
+				)
+				(hide yes)
+			)
+		)
+		(pin "3"
+		)
+		(pin "1"
+		)
+		(pin "4"
+		)
+		(pin "2"
+		)
+		(instances
+			(project "load_automatisation"
+				(path "/e193aeee-7d8e-4a61-b3f1-51249c7839f9"
+					(reference "TENG_Connector2")
+					(unit 1)
+				)
