File: Project/2_Loads.kicad_sch (KiCad schematic)
At the start: 3 parts, among them IC4 MC74VHC138DR2G, IC6 TD62083AFGNEL, IC7 TD62083AFGNEL

Commit message: routing 11/12
Parts:
- added C11, C12, C14: 100nF, Capacitor_SMD:C_0805_2012Metric, symbol Device:C
- added R5: R, Resistor_SMD:R_0805_2012Metric, symbol Device:R
Connections:
- net GND: now also C11.2, C12.2, C14.2
- net VCC: now also R5.2; no longer IC4.16 (VCC), IC6.10 (COMMON), IC7.10 (COMMON)
- new net VCC2: C11.1, C12.1, C14.1, IC4.16 (VCC), IC6.10 (COMMON), IC7.10 (COMMON), R5.1

Commit message: new routing 12/12
Parts:
- IC6, IC7: footprint SOIC127P1030X245-18N -> SamacSys_Parts:SOIC127P1030X245-18N
Changed lines of the file:
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@@
 			)
 		)
-		(property "Footprint" "SOIC127P1030X245-18N"
+		(property "Footprint" "SamacSys_Parts:SOIC127P1030X245-18N"
 			(at 190.5 124.13 0)
 			(effects
@@
 			)
 		)
-		(property "Footprint" "SOIC127P1030X245-18N"
+		(property "Footprint" "SamacSys_Parts:SOIC127P1030X245-18N"
 			(at 138.43 124.13 0)
 			(effects
