File: Project/3_Loads.kicad_sch (KiCad schematic)
At the start: 3 parts, among them IC10 TD62083AFGNEL, IC5 MC74VHC138DR2G, IC8 TD62083AFGNEL

Commit message: routing 11/12
Parts:
- added C10, C13, C8: 100nF, Capacitor_SMD:C_0805_2012Metric, symbol Device:C
- added R6: R, Resistor_SMD:R_0805_2012Metric, symbol Device:R
Connections:
- net GND: now also C10.2, C13.2, C8.2
- net VCC: now also R6.2; no longer IC10.10 (COMMON), IC5.16 (VCC), IC8.10 (COMMON)
- new net VCC3: C10.1, C13.1, C8.1, IC10.10 (COMMON), IC5.16 (VCC), IC8.10 (COMMON), R6.1

Commit message: new routing 12/12
Parts:
- IC10, IC8: footprint SOIC127P1030X245-18N -> SamacSys_Parts:SOIC127P1030X245-18N
Changed lines of the file:
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@@
 			)
 		)
-		(property "Footprint" "SOIC127P1030X245-18N"
+		(property "Footprint" "SamacSys_Parts:SOIC127P1030X245-18N"
 			(at 205.74 140.64 0)
 			(effects
@@
 			)
 		)
-		(property "Footprint" "SOIC127P1030X245-18N"
+		(property "Footprint" "SamacSys_Parts:SOIC127P1030X245-18N"
 			(at 149.86 140.64 0)
 			(effects
